File: Adafruit PCF8523 RTC.sch (EAGLE design)
At the start: 13 parts, among them IC1 RTC_PCF8523T, Q1 32.768

Commit message: https://github.com/adafruit/Adafruit-PCF8523-RTC-Breakout-PCB/issues/1
Parts:
- added C2: 10uF, microbuilder:CAP_CERAMIC0805-NOOUTLINE
- added R3: 1K, microbuilder:RESISTOR0805_NOOUTLINE
- C1: value 0.1uF -> 10uF
Connections:
- new net N$3: C1.1, IC1.VDD, R3.2
- net GND: now also C2.2
- net VCC: now also C2.1, R3.1; no longer C1.1, IC1.VDD
Other:
- moved on the sheet: C1
